Commit message: feat: Add batch retargeting script for lower-body biomechanics using PyRoki
- Implemented a new script `batch_retarget_to_smpl_lower_body.py` for retargeting lower-body biomechanics keypoints.
- Integrated JAX and PyRoki for efficient computation and retargeting.
- Added functions for loading motion data, saving contact labels, and solving retargeting.
- Introduced a shell script `setup_pyroki_env.sh` for setting up a virtual environment and installing dependencies for PyRoki.

File: protomotions/data/assets/urdf/for_retargeting/smpl_humanoid_lower_body_subject_S_GENERIC.urdf (robot description, URDF)
Before this commit: robot smpl_humanoid_lower_body_subject_S_GENERIC, 25 links, 24 joints
Joints:
- joint L_Ankle_x: limit lower=-6.283185 upper=6.283185 effort=500 velocity=100 -> lower=-0.174533 upper=0.174533 effort=500 velocity=100
- joint L_Ankle_y: limit lower=-6.283185 upper=6.283185 effort=500 velocity=100 -> lower=-0.785398 upper=0.349066 effort=500 velocity=100
- joint L_Ankle_z: limit lower=-6.283185 upper=6.283185 effort=500 velocity=100 -> lower=-0.174533 upper=0.174533 effort=500 velocity=100
- joint L_Hip_x: limit lower=-6.283185 upper=6.283185 effort=500 velocity=100 -> lower=-0.349066 upper=0.785398 effort=500 velocity=100
- joint L_Hip_y: limit lower=-6.283185 upper=6.283185 effort=500 velocity=100 -> lower=-0.523599 upper=2.094395 effort=500 velocity=100
- joint L_Hip_z: limit lower=-6.283185 upper=6.283185 effort=500 velocity=100 -> lower=-0.785398 upper=0.785398 effort=500 velocity=100
- joint L_Knee_x: limit lower=-6.283185 upper=6.283185 effort=500 velocity=100 -> lower=-0.174533 upper=0.174533 effort=500 velocity=100
- joint L_Knee_y: limit lower=-6.283185 upper=6.283185 effort=500 velocity=100 -> lower=-0.174533 upper=2.617994 effort=500 velocity=100
- joint L_Knee_z: limit lower=-6.283185 upper=6.283185 effort=500 velocity=100 -> lower=-0.261799 upper=0.261799 effort=500 velocity=100
- joint L_Toe_x: limit lower=-6.283185 upper=6.283185 effort=500 velocity=100 -> lower=-0.174533 upper=0.174533 effort=500 velocity=100
- joint L_Toe_y: limit lower=-6.283185 upper=6.283185 effort=500 velocity=100 -> lower=-0.349066 upper=0.349066 effort=500 velocity=100
- joint L_Toe_z: limit lower=-6.283185 upper=6.283185 effort=500 velocity=100 -> lower=-0.087266 upper=0.087266 effort=500 velocity=100
- joint R_Ankle_x: limit lower=-6.283185 upper=6.283185 effort=500 velocity=100 -> lower=-0.436332 upper=0.436332 effort=500 velocity=100
- joint R_Ankle_y: limit lower=-6.283185 upper=6.283185 effort=500 velocity=100 -> lower=-0.785398 upper=0.349066 effort=500 velocity=100
- joint R_Ankle_z: limit lower=-6.283185 upper=6.283185 effort=500 velocity=100 -> lower=-0.174533 upper=0.174533 effort=500 velocity=100
- joint R_Hip_x: limit lower=-6.283185 upper=6.283185 effort=500 velocity=100 -> lower=-0.349066 upper=0.785398 effort=500 velocity=100
- joint R_Hip_y: limit lower=-6.283185 upper=6.283185 effort=500 velocity=100 -> lower=-0.523599 upper=2.094395 effort=500 velocity=100
- joint R_Hip_z: limit lower=-6.283185 upper=6.283185 effort=500 velocity=100 -> lower=-0.261799 upper=0.261799 effort=500 velocity=100
- joint R_Knee_x: limit lower=-6.283185 upper=6.283185 effort=500 velocity=100 -> lower=-0.174533 upper=0.174533 effort=500 velocity=100
- joint R_Knee_y: limit lower=-6.283185 upper=6.283185 effort=500 velocity=100 -> lower=-0.174533 upper=2.617994 effort=500 velocity=100
- joint R_Knee_z: limit lower=-6.283185 upper=6.283185 effort=500 velocity=100 -> lower=-0.261799 upper=0.261799 effort=500 velocity=100
- joint R_Toe_x: limit lower=-6.283185 upper=6.283185 effort=500 velocity=100 -> lower=-0.174533 upper=0.174533 effort=500 velocity=100
- joint R_Toe_y: limit lower=-6.283185 upper=6.283185 effort=500 velocity=100 -> lower=-0.349066 upper=0.349066 effort=500 velocity=100
- joint R_Toe_z: limit lower=-6.283185 upper=6.283185 effort=500 velocity=100 -> lower=-0.087266 upper=0.087266 effort=500 velocity=100
