Commit message: Add S_GENERIC retargeting and Newton simulator updates

File: protomotions/data/assets/urdf/for_retargeting/smpl_humanoid_lower_body_subject_H170.urdf (robot description, URDF)
Before this commit: robot smpl_humanoid_lower_body_subject_S_GENERIC, 25 links, 24 joints
Joints:
- joint L_Ankle_x: origin xyz=0.000000 0.000000 -0.388300 rpy=0 0 0 -> xyz=0.000000 0.000000 -0.398200 rpy=0 0 0
- joint L_Hip_x: origin xyz=-0.006666 0.095000 -0.092606 rpy=0 0 0 -> xyz=-0.006550 0.095000 -0.091000 rpy=0 0 0
- joint L_Knee_x: origin xyz=-0.006818 0.000000 -0.405700 rpy=0 0 0 -> xyz=-0.006700 0.000000 -0.378900 rpy=0 0 0
- joint L_Toe_x: origin xyz=0.131000 0.000000 -0.055971 rpy=0 0 0 -> xyz=0.123300 0.000000 -0.055000 rpy=0 0 0
- joint R_Ankle_x: origin xyz=0.000000 0.000000 -0.382600 rpy=0 0 0 -> xyz=0.000000 0.000000 -0.398200 rpy=0 0 0
- joint R_Hip_x: origin xyz=-0.006666 -0.095000 -0.092606 rpy=0 0 0 -> xyz=-0.006550 -0.095000 -0.091000 rpy=0 0 0
- joint R_Knee_x: origin xyz=-0.006818 0.000000 -0.408800 rpy=0 0 0 -> xyz=-0.006700 0.000000 -0.378900 rpy=0 0 0
- joint R_Toe_x: origin xyz=0.134200 0.000000 -0.055971 rpy=0 0 0 -> xyz=0.123300 0.000000 -0.055000 rpy=0 0 0
